File: Sistem Mikrokontroler/Tugas 3/Rangkaian Sistem Minimum/Skematik Sistem Minimum.brd (EAGLE design)
At the start: 100 x 80 mm, 16 parts, among them IC2 78L05Z, U1 328P

Commit message: Update Tugas 3
Parts:
- moved S1 29.0 mm to (72.4, 57.1), turned to 90 degrees
- moved C3 18.1 mm to (53.3, 36.8)
- moved C1 16.1 mm to (22.9, 7.62)
- moved R1 5.68 mm to (54.6, 55.9)
- moved Q1 5.08 mm to (20.3, 15.2)
- moved R2 2.54 mm to (38.1, 57.1)
Routing:
- net N$34: track 0.00 -> 80.4 mm
- net N$37: track 0.00 -> 43.0 mm
- net N$2: track 8.15 -> 45.4 mm
- net GND: track 45.0 -> 62.3 mm
- net N$3: track 52.9 -> 60.1 mm
- net VCC: track 73.0 -> 79.4 mm
- net N$36: track 6.65 -> 4.85 mm
Other:
- board text added: "RAMAH X IKI"
